File: hardware/v0.1a/icedemo.kicad_pcb (KiCad board)
At the start: 0 parts

Commit message: Improved schematic and started layout.
* Added inline termination resistors.
* Corrected a mistake in the encoder symbol.
  (Pin 15/13 and missing Pin 70)
* Preliminary positioning of the parts on the PCB.
* Started routing the input data pins.
Parts:
- added A1: iCEBreaker_Bitsy, pkl_module:iCEBreaker_Bitsy, F.Cu at (65.7, 49.4)
- added C1: 100n, pkl_dipol:C_0402, F.Cu at (48.9, 57.5)
- added C10: 100n, pkl_dipol:C_0402, F.Cu at (93.0, 58.0)
- added C11: 100n, pkl_dipol:C_0402, F.Cu at (90.3, 58.0)
- added C12: 100n, pkl_dipol:C_0402, F.Cu at (87.5, 58.0)
- added C13: 100n, pkl_dipol:C_0402, F.Cu at (80.7, 49.4)
- added C14: 100n, pkl_dipol:C_0402, F.Cu at (88.0, 42.9)
- added C15: 100n, pkl_dipol:C_0402, F.Cu at (91.1, 42.9)
- added C16: 10u, pkl_dipol:C_0603, F.Cu at (84.5, 42.8)
- added C17: 100n, pkl_dipol:C_0402, F.Cu at (89.4, 58.0)
- added C18: 100n, pkl_dipol:C_0402, F.Cu at (80.7, 45.8)
- added C19: 100n, pkl_dipol:C_0402, F.Cu at (92.0, 42.9)
- added C2: 100n, pkl_dipol:C_0402, F.Cu at (51.6, 45.2)
- added C20: 10u, pkl_dipol:C_0603, F.Cu at (83.9, 58.2)
- added C21: 100n, pkl_dipol:C_0402, F.Cu at (96.2, 49.0)
- added C22: 100n, pkl_dipol:C_0402, F.Cu at (96.2, 51.9)
- added C23: 10u, pkl_dipol:C_0603, F.Cu at (96.5, 43.1)
- added C24: 10u, pkl_dipol:C_0603, F.Cu at (96.5, 40.9)
- added C25: 10u, pkl_dipol:C_0603, F.Cu at (96.5, 39.6)
- added C3: 100n, pkl_dipol:C_0402, F.Cu at (51.3, 50.1)
- added C4: 100n, pkl_dipol:C_0402, F.Cu at (51.1, 49.4)
- added C5: 100n, pkl_dipol:C_0402, F.Cu at (50.8, 55.5)
- added C6: 100n, pkl_dipol:C_0402, F.Cu at (51.6, 46.4)
- added C7: 4u7, pkl_dipol:C_0603, F.Cu at (85.2, 36.0)
- added C8: 10u, pkl_dipol:C_0603, F.Cu at (87.5, 39.0)
- added C9: 6p8, pkl_dipol:C_0402, F.Cu at (85.2, 38.2)
- added J1: SNES, pkl_connectors:SNES, F.Cu at (36.2, 63.4)
- added J2: HDMI_A, pkl_connectors:HDMI-10029449-111RLF, F.Cu at (102.5, 50.9)
- added L1: 2u2, pkl_dipol:L_0805, F.Cu at (91.4, 36.4)
- added L2: 600, pkl_dipol:L_0402, F.Cu at (86.0, 42.8)
- added L3: 600, pkl_dipol:L_0402, F.Cu at (85.5, 58.2)
- added L4: 600, pkl_dipol:L_0402, F.Cu at (96.5, 42.0)
- added R1: 10k, pkl_dipol:R_0402, F.Cu at (51.0, 56.9)
- added R10: 33R, pkl_dipol:R_Array_Convex_4x0402, F.Cu at (80.7, 56.6)
- added R11: 10k, pkl_dipol:R_0402, F.Cu at (90.1, 39.1)
- added R12: 10k, pkl_dipol:R_0402, F.Cu at (92.2, 39.0)
- added R13: 5k1, pkl_dipol:R_0402, F.Cu at (95.4, 54.8)
- added R14: 2k2, pkl_dipol:R_0402, F.Cu at (98.3, 53.6)
- added R15: 2k2, pkl_dipol:R_0402, F.Cu at (98.3, 52.7)
- added R16: 10k, pkl_dipol:R_0402, F.Cu at (98.4, 55.1)
- added R2: 10k, pkl_dipol:R_0402, F.Cu at (51.5, 44.1)
- added R3: 10k, pkl_dipol:R_0402, F.Cu at (51.2, 51.2)
- added R4: 33R, pkl_dipol:R_Array_Convex_4x0402, F.Cu at (80.7, 53.9)
- added R5: 33R, pkl_dipol:R_Array_Convex_4x0402, F.Cu at (80.7, 44.0)
- added R6: 33R, pkl_dipol:R_Array_Convex_4x0402, F.Cu at (80.7, 51.2)
- added R7: 33R, pkl_dipol:R_Array_Convex_4x0402, F.Cu at (80.7, 47.6)
- added R8: 4k7, pkl_dipol:R_0402, F.Cu at (92.9, 42.9)
- added R9: 4k7, pkl_dipol:R_0402, F.Cu at (93.8, 42.9)
- added SW1: TACT, pkl_buttons_switches:SW_SPST_3x4x2.5, F.Cu at (50.5, 67.5)
- added U1: 74LVC2T45, pkl_housings_sot:SOT-833-1, F.Cu at (48.9, 55.2)
- added U2: 74LVC2T45, pkl_housings_sot:SOT-833-1, F.Cu at (49.2, 45.4)
- added U3: 74LVC2T45, pkl_housings_sot:SOT-833-1, F.Cu at (48.9, 50.5)
- added U4: SII902xA-mod, Package_DFN_QFN:QFN-72-1EP_10x10mm_P0.5mm_EP6x6mm_ThermalVias, F.Cu at (89.2, 50.1)
- added U5: TLV62568DBV, pkl_housings_sot:SOT-23-5, F.Cu at (87.7, 36.4)
Routing:
- net Net-(R5-Pad4): track 0.00 -> 4.36 mm
- net /CVCC12: track 0.00 -> 4.00 mm, vias 0 -> 1
- net Net-(R10-Pad5): track 0.00 -> 3.87 mm
- net Net-(R10-Pad7): track 0.00 -> 3.83 mm
- net Net-(R5-Pad6): track 0.00 -> 3.75 mm
- net Net-(R5-Pad8): track 0.00 -> 3.70 mm
- net Net-(R4-Pad8): track 0.00 -> 3.62 mm
- net Net-(R4-Pad6): track 0.00 -> 3.58 mm
- net Net-(R4-Pad4): track 0.00 -> 3.58 mm
- net Net-(R4-Pad2): track 0.00 -> 3.54 mm
- net /IOVCC: track 0.00 -> 3.52 mm
- net Net-(R7-Pad2): track 0.00 -> 3.33 mm
- net Net-(R6-Pad8): track 0.00 -> 3.33 mm
- net Net-(R6-Pad6): track 0.00 -> 3.29 mm
- net Net-(R6-Pad4): track 0.00 -> 3.29 mm
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Other:
- board outline added: 80 x 40 mm
- copper layers 0 -> 4
